File: embedded-debug/embedded-debug.kicad_pcb (KiCad board)
At the start: 2 copper layers, 50.8 x 24.1 mm, 23 parts, among them J1 Conn_02x05_Odd_Even, J2 Conn_02x05_Odd_Even, J3 Conn_01x02, J4 USB_C_Receptacle_USB2.0, J5 AVR-ISP-6, J6 Conn_02x05_Odd_Even, SW1 SW_Push, U1 FT230XQ

Commit message: Committing and order rev-1
Routing:
- net GND: track 23.4 -> 24.7 mm
Other:
- board text added: "rev-1"
